Commit message: put the ground on the ground

File: go2_robot_sdk/urdf/go2.urdf (robot description, URDF)
Before this commit: robot go2, 33 links, 32 joints
Joints:
- joint base_footprint_joint: origin xyz=0 0 0 rpy=0 0 0 -> xyz=0 0 -0.32 rpy=0 0 0

Commit message: undo making the ground the ground

File: go2_robot_sdk/urdf/go2.urdf (robot description, URDF)
Before this commit: robot go2, 33 links, 32 joints
Joints:
- joint base_footprint_joint: origin xyz=0 0 -0.32 rpy=0 0 0 -> xyz=0 0 0 rpy=0 0 0
